File: 65-wkl-pcb/65-wkl-pcb.kicad_pcb (KiCad board)
At the start: 2 copper layers, 160 parts, among them J3 Conn_01x05, J4 Conn_01x04, U3 RP2040, U4 W25Q128JVS, Y1 Crystal_GND24

Commit message: PCB
Parts:
- added C1: 1u, Capacitor_SMD:C_0402_1005Metric, B.Cu at (104.8, 50.8)
- added C2: 1u, Capacitor_SMD:C_0402_1005Metric, B.Cu at (102.3, 56.4)
- added U1: XC6206PxxxMR, Package_TO_SOT_SMD:SOT-23-3, B.Cu at (102.3, 53.2)
- J3: footprint Connector_PinSocket_2.54mm:PinSocket_1x05_P2.54mm_Vertical -> Connector_PinHeader_2.54mm:PinHeader_1x05_P2.54mm_Vertical
- J4: footprint Connector_JST:JST_PH_S4B-PH-K_1x04_P2.00mm_Horizontal -> Connector_Molex:Molex_Pico-EZmate_78171-0004_1x04-1MP_P1.20mm_Vertical
- moved J4 89.8 mm to (119.9, 50.8), turned to 0 degrees
- moved R3 64.6 mm to (130.4, 71.8)
- moved BOOT1 62.4 mm to (136.4, 72.4)
- moved R4 61.0 mm to (130.4, 73.0), turned to 0 degrees
- moved R6 59.9 mm to (118.4, 102.5), turned to -90 degrees
- moved R5 58.1 mm to (130.4, 74.2)
- moved C5 55.1 mm to (112.7, 79.4)
- moved RST1 53.3 mm to (113.5, 101.6)
- moved C16 52.2 mm to (128.2, 87.6)
- moved C13 52.2 mm to (129.2, 87.6)
- moved R8 52.2 mm to (126.1, 87.6)
- moved R7 52.2 mm to (127.2, 87.6)
- moved R9 51.5 mm to (128.9, 104.1), turned to 90 degrees
- moved Y1 51.5 mm to (131.2, 105.8)
- moved C11 51.5 mm to (133.1, 107.6)
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Connections:
- D1 pad 1: unconnected-(D1-K-Pad1) -> ROW0
- D10 pad 1: unconnected-(D10-K-Pad1) -> ROW0
- D11 pad 1: unconnected-(D11-K-Pad1) -> ROW0
- D12 pad 1: unconnected-(D12-K-Pad1) -> ROW0
- D13 pad 1: unconnected-(D13-K-Pad1) -> ROW0
- D14 pad 1: unconnected-(D14-K-Pad1) -> ROW0
- D15 pad 1: unconnected-(D15-K-Pad1) -> ROW1
- D16 pad 1: unconnected-(D16-K-Pad1) -> ROW1
- D17 pad 1: unconnected-(D17-K-Pad1) -> ROW1
- D18 pad 1: unconnected-(D18-K-Pad1) -> ROW1
- D19 pad 1: unconnected-(D19-K-Pad1) -> ROW1
- D2 pad 1: unconnected-(D2-K-Pad1) -> ROW0
- D20 pad 1: unconnected-(D20-K-Pad1) -> ROW1
- D21 pad 1: unconnected-(D21-K-Pad1) -> ROW1
- D22 pad 1: unconnected-(D22-K-Pad1) -> ROW1
- D23 pad 1: unconnected-(D23-K-Pad1) -> ROW1
- D24 pad 1: unconnected-(D24-K-Pad1) -> ROW1
- D25 pad 1: unconnected-(D25-K-Pad1) -> ROW1
- D26 pad 1: unconnected-(D26-K-Pad1) -> ROW1
- D27 pad 1: unconnected-(D27-K-Pad1) -> ROW1
- D28 pad 1: unconnected-(D28-K-Pad1) -> ROW1
- D29 pad 1: unconnected-(D29-K-Pad1) -> ROW1
- D3 pad 1: unconnected-(D3-K-Pad1) -> ROW0
- D30 pad 1: unconnected-(D30-K-Pad1) -> ROW2
- D31 pad 1: unconnected-(D31-K-Pad1) -> ROW2
- D32 pad 1: unconnected-(D32-K-Pad1) -> ROW2
- D33 pad 1: unconnected-(D33-K-Pad1) -> ROW2
- D34 pad 1: unconnected-(D34-K-Pad1) -> ROW2
- D35 pad 1: unconnected-(D35-K-Pad1) -> ROW2
- D36 pad 1: unconnected-(D36-K-Pad1) -> ROW2
- D37 pad 1: unconnected-(D37-K-Pad1) -> ROW2
- D38 pad 1: unconnected-(D38-K-Pad1) -> ROW2
- D39 pad 1: unconnected-(D39-K-Pad1) -> ROW2
- D4 pad 1: unconnected-(D4-K-Pad1) -> ROW0
- D40 pad 1: unconnected-(D40-K-Pad1) -> ROW2
- D41 pad 1: unconnected-(D41-K-Pad1) -> ROW2
- D42 pad 1: unconnected-(D42-K-Pad1) -> ROW2
- D43 pad 1: unconnected-(D43-K-Pad1) -> ROW2
- D44 pad 1: unconnected-(D44-K-Pad1) -> ROW3
- D45 pad 1: unconnected-(D45-K-Pad1) -> ROW3
- D46 pad 1: unconnected-(D46-K-Pad1) -> ROW3
- D47 pad 1: unconnected-(D47-K-Pad1) -> ROW3
- D48 pad 1: unconnected-(D48-K-Pad1) -> ROW3
- D49 pad 1: unconnected-(D49-K-Pad1) -> ROW3
- D5 pad 1: unconnected-(D5-K-Pad1) -> ROW0
- D50 pad 1: unconnected-(D50-K-Pad1) -> ROW3
- D51 pad 1: unconnected-(D51-K-Pad1) -> ROW3
- D52 pad 1: unconnected-(D52-K-Pad1) -> ROW3
- D53 pad 1: unconnected-(D53-K-Pad1) -> ROW3
- D54 pad 1: unconnected-(D54-K-Pad1) -> ROW3
- D55 pad 1: unconnected-(D55-K-Pad1) -> ROW3
- D56 pad 1: unconnected-(D56-K-Pad1) -> ROW3
- D57 pad 1: unconnected-(D57-K-Pad1) -> ROW3
- D58 pad 1: unconnected-(D58-K-Pad1) -> ROW4
- D59 pad 1: unconnected-(D59-K-Pad1) -> ROW4
- D6 pad 1: unconnected-(D6-K-Pad1) -> ROW0
- D60 pad 1: unconnected-(D60-K-Pad1) -> ROW4
- D61 pad 1: unconnected-(D61-K-Pad1) -> ROW4
- D62 pad 1: unconnected-(D62-K-Pad1) -> ROW4
- D63 pad 1: unconnected-(D63-K-Pad1) -> ROW4
- D64 pad 1: unconnected-(D64-K-Pad1) -> ROW4
- D7 pad 1: unconnected-(D7-K-Pad1) -> ROW0
- D8 pad 1: unconnected-(D8-K-Pad1) -> ROW0
- D9 pad 1: unconnected-(D9-K-Pad1) -> ROW0
- J3 pad 1: RESET -> SWC
- J3 pad 2: +3V3 -> SWD
- J3 pad 3: GND -> RESET
- J3 pad 4: SWC -> +3V3
- J3 pad 5: SWD -> GND
- MX1 pad 1: unconnected-(MX1-Pad1) -> COL0
- MX10 pad 1: unconnected-(MX10-Pad1) -> COL9
- MX11 pad 1: unconnected-(MX11-Pad1) -> COL10
- MX12 pad 1: unconnected-(MX12-Pad1) -> COL11
- MX13 pad 1: unconnected-(MX13-Pad1) -> COL12
- MX14 pad 1: unconnected-(MX14-Pad1) -> COL13
- MX15 pad 1: unconnected-(MX15-Pad1) -> COL0
- MX16 pad 1: unconnected-(MX16-Pad1) -> COL1
- MX17 pad 1: unconnected-(MX17-Pad1) -> COL2
- MX18 pad 1: unconnected-(MX18-Pad1) -> COL3
- MX19 pad 1: unconnected-(MX19-Pad1) -> COL4
- MX2 pad 1: unconnected-(MX2-Pad1) -> COL1
- MX20 pad 1: unconnected-(MX20-Pad1) -> COL5
- MX21 pad 1: unconnected-(MX21-Pad1) -> COL6
- MX22 pad 1: unconnected-(MX22-Pad1) -> COL7
- MX23 pad 1: unconnected-(MX23-Pad1) -> COL8
- MX24 pad 1: unconnected-(MX24-Pad1) -> COL9
- MX25 pad 1: unconnected-(MX25-Pad1) -> COL10
- MX26 pad 1: unconnected-(MX26-Pad1) -> COL11
- MX27 pad 1: unconnected-(MX27-Pad1) -> COL12
- MX28 pad 1: unconnected-(MX28-Pad1) -> COL13
- MX29 pad 1: unconnected-(MX29-Pad1) -> Net-(MX29-Pad1)
- MX3 pad 1: unconnected-(MX3-Pad1) -> COL2
- MX30 pad 1: unconnected-(MX30-Pad1) -> COL0
- MX31 pad 1: unconnected-(MX31-Pad1) -> COL1
- MX32 pad 1: unconnected-(MX32-Pad1) -> COL2
- MX33 pad 1: unconnected-(MX33-Pad1) -> COL3
- MX34 pad 1: unconnected-(MX34-Pad1) -> COL4
- MX35 pad 1: unconnected-(MX35-Pad1) -> COL5
- MX36 pad 1: unconnected-(MX36-Pad1) -> COL6
- MX37 pad 1: unconnected-(MX37-Pad1) -> COL7
- MX38 pad 1: unconnected-(MX38-Pad1) -> COL8
- MX39 pad 1: unconnected-(MX39-Pad1) -> COL9
- MX4 pad 1: unconnected-(MX4-Pad1) -> COL3
- MX40 pad 1: unconnected-(MX40-Pad1) -> COL10
- MX41 pad 1: unconnected-(MX41-Pad1) -> COL11
- MX42 pad 1: unconnected-(MX42-Pad1) -> COL13
- MX43 pad 1: unconnected-(MX43-Pad1) -> Net-(MX29-Pad1)
- MX44 pad 1: unconnected-(MX44-Pad1) -> COL0
- MX45 pad 1: unconnected-(MX45-Pad1) -> COL1
- MX46 pad 1: unconnected-(MX46-Pad1) -> COL2
- MX47 pad 1: unconnected-(MX47-Pad1) -> COL3
- MX48 pad 1: unconnected-(MX48-Pad1) -> COL4
- MX49 pad 1: unconnected-(MX49-Pad1) -> COL5
- MX5 pad 1: unconnected-(MX5-Pad1) -> COL4
- MX50 pad 1: unconnected-(MX50-Pad1) -> COL6
- MX51 pad 1: unconnected-(MX51-Pad1) -> COL7
- MX52 pad 1: unconnected-(MX52-Pad1) -> COL8
- MX53 pad 1: unconnected-(MX53-Pad1) -> COL9
- MX54 pad 1: unconnected-(MX54-Pad1) -> COL10
- MX55 pad 1: unconnected-(MX55-Pad1) -> COL11
- MX56 pad 1: unconnected-(MX56-Pad1) -> COL13
- MX57 pad 1: unconnected-(MX57-Pad1) -> Net-(MX29-Pad1)
- MX58 pad 1: unconnected-(MX58-Pad1) -> COL0
- MX59 pad 1: unconnected-(MX59-Pad1) -> COL2
- MX6 pad 1: unconnected-(MX6-Pad1) -> COL5
- MX60 pad 1: unconnected-(MX60-Pad1) -> COL5
- MX61 pad 1: unconnected-(MX61-Pad1) -> COL10
- MX62 pad 1: unconnected-(MX62-Pad1) -> COL12
- MX63 pad 1: unconnected-(MX63-Pad1) -> COL13
- MX64 pad 1: unconnected-(MX64-Pad1) -> Net-(MX29-Pad1)
- MX7 pad 1: unconnected-(MX7-Pad1) -> COL6
- MX8 pad 1: unconnected-(MX8-Pad1) -> COL7
- MX9 pad 1: unconnected-(MX9-Pad1) -> COL8
- R4 pad 1: Net-(R4-Pad1) -> Q_SEL
- R5 pad 2: Net-(R4-Pad1) -> Q_SEL
Routing:
- net ROW1: track 0.00 -> 408.0 mm
- net ROW0: track 0.00 -> 398.8 mm
- net ROW2: track 0.00 -> 386.8 mm, vias 0 -> 2
- net ROW3: track 0.00 -> 286.3 mm, vias 0 -> 4
- net ROW4: track 0.00 -> 285.0 mm, vias 0 -> 4
- net COL13: track 0.00 -> 235.3 mm
- net Net-(MX29-Pad1): track 0.00 -> 224.8 mm
- net COL12: track 0.00 -> 215.5 mm
- net COL10: track 0.00 -> 178.9 mm
- net +3V3: track 0.00 -> 162.0 mm, vias 0 -> 4
- net COL0: track 0.00 -> 144.8 mm
- net COL2: track 0.00 -> 127.5 mm
- net GND: track 0.00 -> 105.1 mm, vias 0 -> 23
- net COL4: track 0.00 -> 105.0 mm, vias 0 -> 2
- net COL5: track 0.00 -> 104.0 mm
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- added copper zone on B.Cu, net GND
- added copper zone on F.Cu, net GND
Other:
- board outline added: 303.2 x 93.7 mm

Commit message: production
Parts:
- added G***: LOGO, LOGO, F.Cu at (310.4, 24.6)
- added G***: LOGO, LOGO, F.Cu at (175.4, 100.0)
- added G***: LOGO, LOGO, B.Cu at (310.0, 24.6)
- added G***: LOGO, LOGO, B.Cu at (308.8, 51.6)
Connections:
- MX29 pad 1: Net-(MX29-Pad1) -> COL14
- MX43 pad 1: Net-(MX29-Pad1) -> COL14
- MX57 pad 1: Net-(MX29-Pad1) -> COL14
- MX64 pad 1: Net-(MX29-Pad1) -> COL14
- U3 pad 12: unconnected-(U3-GPIO9-Pad12) -> COL8
- U3 pad 13: unconnected-(U3-GPIO10-Pad13) -> COL14
- U3 pad 14: unconnected-(U3-GPIO11-Pad14) -> COL13
- U3 pad 15: unconnected-(U3-GPIO12-Pad15) -> COL12
- U3 pad 16: unconnected-(U3-GPIO13-Pad16) -> COL10
- U3 pad 17: unconnected-(U3-GPIO14-Pad17) -> COL5
- U3 pad 18: unconnected-(U3-GPIO15-Pad18) -> ROW4
- U3 pad 27: unconnected-(U3-GPIO16-Pad27) -> COL2
- U3 pad 28: unconnected-(U3-GPIO17-Pad28) -> COL0
- U3 pad 29: unconnected-(U3-GPIO18-Pad29) -> ROW0
- U3 pad 30: unconnected-(U3-GPIO19-Pad30) -> ROW1
- U3 pad 31: unconnected-(U3-GPIO20-Pad31) -> ROW2
- U3 pad 35: unconnected-(U3-GPIO23-Pad35) -> COL1
- U3 pad 36: unconnected-(U3-GPIO24-Pad36) -> ROW3
- U3 pad 37: unconnected-(U3-GPIO25-Pad37) -> COL3
- U3 pad 38: unconnected-(U3-GPIO26_ADC0-Pad38) -> COL4
- U3 pad 5: unconnected-(U3-GPIO3-Pad5) -> COL7
- U3 pad 6: unconnected-(U3-GPIO4-Pad6) -> COL6
- U3 pad 7: unconnected-(U3-GPIO5-Pad7) -> COL11
- U3 pad 8: unconnected-(U3-GPIO6-Pad8) -> COL9
Routing:
- net COL14: track 0.00 -> 238.4 mm
- net Net-(MX29-Pad1): track 224.8 -> 0.00 mm
- net COL1: track 46.0 -> 214.6 mm
- net COL11: track 70.0 -> 217.7 mm
- net COL6: track 67.0 -> 180.1 mm
- net COL9: track 67.0 -> 169.4 mm
- net COL7: track 67.0 -> 159.5 mm
- net COL8: track 67.0 -> 147.7 mm
- net COL0: track 144.8 -> 188.2 mm
- net ROW2: track 386.8 -> 417.2 mm
- net ROW0: track 398.8 -> 428.4 mm
- net ROW1: track 408.0 -> 434.3 mm
- net COL2: track 127.5 -> 140.7 mm
- net COL13: track 235.3 -> 248.1 mm
- net COL12: track 215.5 -> 228.0 mm
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Other:
- board text added: "BOOT"
- board text added: "HKL 2024"
- board text added: "RST"

Commit message: layout
Parts:
- MX61: footprint PCM_marbastlib-mx:SW_MX_1.5u -> PCM_marbastlib-mx:SW_MX_1u
- S1: footprint PCM_marbastlib-mx:STAB_MX_P_6.25u -> PCM_marbastlib-mx:STAB_MX_P_7u
- moved D61 4.76 mm to (237.3, 101.6)
- moved D59 4.76 mm to (80.2, 101.6)
- moved MX59 4.76 mm to (77.0, 100.8)
- moved MX61 4.76 mm to (234.2, 100.8)
- moved S1 2.39 mm to (158.0, 101.0)
- moved MX60 2.38 mm to (158.0, 100.8)
- moved D60 2.38 mm to (161.1, 101.6)
Routing:
- net COL2: track 140.7 -> 147.4 mm
- net COL5: track 115.5 -> 118.9 mm
- net COL10: track 190.8 -> 193.6 mm
- net Net-(D60-A): track 3.59 -> 4.22 mm
- net COL12: track 228.0 -> 228.6 mm
- net COL13: track 248.1 -> 248.7 mm
- net COL8: track 147.7 -> 148.3 mm
- net COL7: track 159.5 -> 160.1 mm
- net COL6: track 180.1 -> 180.7 mm
- net COL14: track 238.4 -> 239.0 mm
- net COL9: track 169.4 -> 170.0 mm
- net COL11: track 217.7 -> 218.3 mm
