File: 65-wkl-pcb/65-wkl-pcb.kicad_sch (KiCad schematic)
At the start: 160 parts, among them J3 Conn_01x05, J4 Conn_01x04, U3 RP2040, U4 W25Q128JVS, Y1 Crystal_GND24

Commit message: PCB
Parts:
- added C1, C2: 1u, Capacitor_SMD:C_0402_1005Metric, symbol Device:C_Small
- added U1: XC6206PxxxMR, Package_TO_SOT_SMD:SOT-23-3, symbol Regulator_Linear:XC6206PxxxMR
- J3: footprint Connector_PinSocket_2.54mm:PinSocket_1x05_P2.54mm_Vertical -> Connector_PinHeader_2.54mm:PinHeader_1x05_P2.54mm_Vertical
- J4: footprint Connector_JST:JST_PH_S4B-PH-K_1x04_P2.00mm_Horizontal -> Connector_Molex:Molex_Pico-EZmate_78171-0004_1x04-1MP_P1.20mm_Vertical
Connections:
- net +3V3: now also J3.4 (Pin_4), C2.1, U1.2 (VO); no longer J3.2 (Pin_2)
- net +5V: now also C1.1, U1.3 (VI)
- net GND: now also J3.5 (Pin_5), C1.2, C2.2, U1.1 (GND); no longer J3.3 (Pin_3)
- net Q_SEL: now also R4.1, R5.2
- net RESET: now also J3.3 (Pin_3); no longer J3.1 (Pin_1)
- net SWC: now also J3.1 (Pin_1); no longer J3.4 (Pin_4)
- net SWD: now also J3.2 (Pin_2); no longer J3.5 (Pin_5)
- net COL5: now reaches MX49.1
- net COL5: now also MX20.1, MX35.1, MX6.1, MX60.1
- net COL0: now reaches MX58.1
- net COL0: now also MX1.1, MX15.1, MX30.1, MX44.1
- net ROW1: now reaches D15.1 (K)
- net ROW1: now also D16.1 (K), D17.1 (K), D18.1 (K), D19.1 (K), D20.1 (K), D21.1 (K), D22.1 (K), D23.1 (K), D24.1 (K), D25.1 (K), D26.1 (K), D27.1 (K), D28.1 (K), D29.1 (K)
- net COL3: now reaches MX47.1
- net COL3: now also MX18.1, MX33.1, MX4.1
- net ROW3: now reaches D53.1 (K)
- net ROW3: now also D44.1 (K), D45.1 (K), D46.1 (K), D47.1 (K), D48.1 (K), D49.1 (K), D50.1 (K), D51.1 (K), D52.1 (K), D54.1 (K), D55.1 (K), D56.1 (K), D57.1 (K)
- net ROW2: now reaches D35.1 (K)
- net ROW2: now also D30.1 (K), D31.1 (K), D32.1 (K), D33.1 (K), D34.1 (K), D36.1 (K), D37.1 (K), D38.1 (K), D39.1 (K), D40.1 (K), D41.1 (K), D42.1 (K), D43.1 (K)
- net at MX29.1: now also MX43.1, MX57.1, MX64.1
- net COL4: now reaches MX48.1
- net COL4: now also MX19.1, MX34.1, MX5.1
- net ROW0: now reaches D3.1 (K)
- net ROW0: now also D1.1 (K), D10.1 (K), D11.1 (K), D12.1 (K), D13.1 (K), D14.1 (K), D2.1 (K), D4.1 (K), D5.1 (K), D6.1 (K), D7.1 (K), D8.1 (K), D9.1 (K)
- net COL12: now reaches MX13.1
- net COL12: now also MX27.1, MX62.1
- net COL7: now reaches MX37.1
- net COL7: now also MX22.1, MX51.1, MX8.1
- net COL13: now reaches MX28.1
- net COL13: now also MX14.1, MX42.1, MX56.1, MX63.1
- net COL2: now reaches MX46.1
- net COL2: now also MX17.1, MX3.1, MX32.1, MX59.1
- net COL1: now reaches MX31.1
- net COL1: now also MX16.1, MX2.1, MX45.1
- net COL9: now reaches MX39.1
- net COL9: now also MX10.1, MX24.1, MX53.1
- net ROW4: now reaches D62.1 (K)
- net ROW4: now also D58.1 (K), D59.1 (K), D60.1 (K), D61.1 (K), D63.1 (K), D64.1 (K)
- net COL11: now reaches MX26.1
- net COL11: now also MX12.1, MX41.1, MX55.1
- net COL10: now reaches MX25.1
- net COL10: now also MX11.1, MX40.1, MX54.1, MX61.1
- net COL6: now reaches MX50.1
- net COL6: now also MX21.1, MX36.1, MX7.1
- net COL8: now reaches MX9.1
- net COL8: now also MX23.1, MX38.1, MX52.1
Other:
- moved on the sheet: D42, D43, D56, D57, D62, D63, D64, MX42, MX43, MX56, MX57, MX62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

Commit message: bus
Connections:
- net COL0: now also U3.29 (GPIO18)
- net COL13: now also MX29.1, MX43.1, MX57.1, MX64.1
- net COL2: now also U3.30 (GPIO19)
- net COL3: now also U3.36 (GPIO24)
- net COL4: now also U3.37 (GPIO25)
- net COL5: now also U3.17 (GPIO14)
- net ROW0: now also U3.31 (GPIO20)
- net ROW1: now also U3.32 (GPIO21)
- net ROW2: now also U3.34 (GPIO22)
- net ROW3: now also U3.35 (GPIO23)
- net ROW4: now also U3.18 (GPIO15)
Changed lines of the file:
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@@
 	)
 	(junction
+		(at 370.84 67.31)
+		(diameter 0)
+		(color 0 0 0 0)
+	)
+	(junction
 		(at 101.6 139.7)
 		(diameter 0)
@@
 	(wire
 		(pts
+			(xy 370.84 35.56) (xy 370.84 67.31)
+		)
+		(stroke
+			(width 0)
+			(type default)
+		)
+	)
+	(wire
+		(pts
 			(xy 194.31 58.42) (xy 208.28 58.42)
 		)
@@
 	(global_label "COL4"
 		(shape input)
-		(at 226.06 158.75 90)
+		(at 76.2 226.06 0)
 		(fields_autoplaced yes)
 		(effects
@@
 		)
 		(property "Intersheetrefs" "${INTERSHEET_REFS}"
-			(at 226.06 150.9267 90)
+			(at 84.0233 226.06 0)
 			(effects
 				(font
@@
 		)
 	)
+	(global_label "COL13"
+		(shape input)
+		(at 370.84 35.56 90)
+		(fields_autoplaced yes)
+		(effects
+			(font
+				(size 1.27 1.27)
+			)
+			(justify left)
+		)
+		(property "Intersheetrefs" "${INTERSHEET_REFS}"
+			(at 370.84 26.5272 90)
+			(effects
+				(font
+					(size 1.27 1.27)
+				)
+				(justify left)
+				(hide yes)
+			)
+		)
+	)
 	(global_label "ROW0"
 		(shape input)
-		(at 158.75 160.02 180)
+		(at 76.2 213.36 0)
 		(fields_autoplaced yes)
 		(effects
@@
 				(size 1.27 1.27)
 			)
-			(justify right)
+			(justify left)
 		)
 		(property "Intersheetrefs" "${INTERSHEET_REFS}"
-			(at 150.5034 160.02 0)
+			(at 84.4466 213.36 0)
 			(effects
 				(font
 					(size 1.27 1.27)
 				)
-				(justify right)
+				(justify left)
 				(hide yes)
 			)
@@
 	(global_label "COL0"
 		(shape input)
-		(at 170.18 158.75 90)
+		(at 76.2 208.28 0)
 		(fields_autoplaced yes)
 		(effects
@@
 		)
 		(property "Intersheetrefs" "${INTERSHEET_REFS}"
-			(at 170.18 150.9267 90)
+			(at 84.0233 208.28 0)
 			(effects
 				(font
@@
 	(global_label "COL3"
 		(shape input)
-		(at 212.09 158.75 90)
+		(at 76.2 223.52 0)
 		(fields_autoplaced yes)
 		(effects
@@
 		)
 		(property "Intersheetrefs" "${INTERSHEET_REFS}"
-			(at 212.09 150.9267 90)
+			(at 84.0233 223.52 0)
 			(effects
 				(font
@@
 	(global_label "COL2"
 		(shape input)
-		(at 198.12 158.75 90)
+		(at 76.2 210.82 0)
 		(fields_autoplaced yes)
 		(effects
@@
 		)
 		(property "Intersheetrefs" "${INTERSHEET_REFS}"
-			(at 198.12 150.9267 90)
+			(at 84.0233 210.82 0)
 			(effects
 				(font
@@
 	(global_label "ROW1"
 		(shape input)
-		(at 158.75 179.07 180)
+		(at 76.2 215.9 0)
 		(fields_autoplaced yes)
 		(effects
@@
 				(size 1.27 1.27)
 			)
-			(justify right)
+			(justify left)
 		)
 		(property "Intersheetrefs" "${INTERSHEET_REFS}"
-			(at 150.5034 179.07 0)
+			(at 84.4466 215.9 0)
 			(effects
 				(font
 					(size 1.27 1.27)
 				)
-				(justify right)
+				(justify left)
 				(hide yes)
 			)
@@
 	(global_label "COL5"
 		(shape input)
-		(at 240.03 158.75 90)
+		(at 76.2 198.12 0)
 		(fields_autoplaced yes)
 		(effects
@@
 		)
 		(property "Intersheetrefs" "${INTERSHEET_REFS}"
-			(at 240.03 150.9267 90)
+			(at 84.0233 198.12 0)
 			(effects
 				(font
@@
 	(global_label "ROW4"
 		(shape input)
-		(at 158.75 236.22 180)
+		(at 76.2 200.66 0)
 		(fields_autoplaced yes)
 		(effects
@@
 				(size 1.27 1.27)
 			)
-			(justify right)
+			(justify left)
 		)
 		(property "Intersheetrefs" "${INTERSHEET_REFS}"
-			(at 150.5034 236.22 0)
+			(at 84.4466 200.66 0)
 			(effects
 				(font
 					(size 1.27 1.27)
 				)
-				(justify right)
+				(justify left)
 				(hide yes)
 			)
@@
 	(global_label "ROW2"
 		(shape input)
-		(at 158.75 198.12 180)
+		(at 76.2 218.44 0)
 		(fields_autoplaced yes)
 		(effects
@@
 				(size 1.27 1.27)
 			)
-			(justify right)
+			(justify left)
 		)
 		(property "Intersheetrefs" "${INTERSHEET_REFS}"
-			(at 150.5034 198.12 0)
+			(at 84.4466 218.44 0)
 			(effects
 				(font
 					(size 1.27 1.27)
 				)
-				(justify right)
+				(justify left)
 				(hide yes)
 			)
@@
 	(global_label "ROW3"
 		(shape input)
-		(at 158.75 217.17 180)
+		(at 76.2 220.98 0)
 		(fields_autoplaced yes)
 		(effects
@@
 				(size 1.27 1.27)
 			)
-			(justify right)
+			(justify left)
 		)
 		(property "Intersheetrefs" "${INTERSHEET_REFS}"
-			(at 150.5034 217.17 0)
+			(at 84.4466 220.98 0)
 			(effects
 				(font
 					(size 1.27 1.27)
 				)
-				(justify right)
+				(justify left)
 				(hide yes)
 			)

Commit message: production
Connections:
- net COL0: now also U3.28 (GPIO17); no longer U3.29 (GPIO18)
- net COL1: now also U3.35 (GPIO23)
- net COL10: now also U3.16 (GPIO13)
- net COL11: now also U3.7 (GPIO5)
- net COL12: now also U3.15 (GPIO12)
- net COL13: now also U3.14 (GPIO11); no longer MX29.1, MX43.1, MX57.1, MX64.1
- net COL2: now also U3.27 (GPIO16); no longer U3.30 (GPIO19)
- net COL3: now also U3.37 (GPIO25); no longer U3.36 (GPIO24)
- net COL4: now also U3.38 (GPIO26_ADC0); no longer U3.37 (GPIO25)
- net COL6: now also U3.6 (GPIO4)
- net COL7: now also U3.5 (GPIO3)
- net COL8: now also U3.12 (GPIO9)
- net COL9: now also U3.8 (GPIO6)
- net ROW0: now also U3.29 (GPIO18); no longer U3.31 (GPIO20)
- net ROW1: now also U3.30 (GPIO19); no longer U3.32 (GPIO21)
- net ROW2: now also U3.31 (GPIO20); no longer U3.34 (GPIO22)
- net ROW3: now also U3.36 (GPIO24); no longer U3.35 (GPIO23)
- net COL14: now reaches U3.13 (GPIO10)
- net COL14: now also MX29.1, MX43.1, MX57.1, MX64.1

Commit message: layout
Parts:
- MX61: footprint PCM_marbastlib-mx:SW_MX_1.5u -> PCM_marbastlib-mx:SW_MX_1u
- S1: footprint PCM_marbastlib-mx:STAB_MX_P_6.25u -> PCM_marbastlib-mx:STAB_MX_P_7u
Changed lines of the file:
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@@
 			)
 		)
-		(property "Footprint" "PCM_marbastlib-mx:STAB_MX_P_6.25u"
+		(property "Footprint" "PCM_marbastlib-mx:STAB_MX_P_7u"
 			(at 267.97 129.54 0)
 			(effects
@@
 			)
 		)
-		(property "Footprint" "PCM_marbastlib-mx:SW_MX_1.5u"
+		(property "Footprint" "PCM_marbastlib-mx:SW_MX_1u"
 			(at 317.5 127 0)
 			(effects
