File: Daughterboard/UDB.kicad_sch (KiCad schematic)
At the start: 13 parts, among them J1 TYPE-C-31-M12_13, J2 X1224WRS-04-LPV01, U1 TPD4E05U06DQAR

Commit message: layout
Parts:
- J1: footprint acheron_Connectors:TYPE-C-31-M-12 -> acheron_Connectors:USB_C_Receptacle_Hroparts_TYPE-C-31-M-12
